Commit message: Complete task-space teleoperation: UR5 master-slave with analytical IK
- Forward kinematics on master arm
- Analytical inverse kinematics on slave (ur-analytic-ik)
- 100Hz control loop
- Position error < 1mm
- RViz visualization with dual UR5 arms

File: src/teleop_description/urdf/arm_6dof.ros2_control.xacro (robot description, xacro)
@@ -3,5 +3,4 @@
   <xacro:macro name="arm_6dof_ros2_control" params="arm_id use_sim:=true">
     <ros2_control name="${arm_id}_controller" type="system">
-      <!-- Hardware interface -->
       <hardware>
         <xacro:if value="${use_sim}">
@@ -9,9 +8,9 @@
         </xacro:if>
       </hardware>
-      <!-- Joint 1 -->
-      <joint name="${arm_id}_joint1">
+      <!-- UR5 Joint Names -->
+      <joint name="${arm_id}_shoulder_pan_joint">
         <command_interface name="position">
-          <param name="min">-3.14159</param>
-          <param name="max">3.14159</param>
+          <param name="min">-6.2832</param>
+          <param name="max">6.2832</param>
         </command_interface>
         <state_interface name="position"/>
@@ -19,9 +18,8 @@
         <state_interface name="effort"/>
       </joint>
-      <!-- Joint 2 -->
-      <joint name="${arm_id}_joint2">
+      <joint name="${arm_id}_shoulder_lift_joint">
         <command_interface name="position">
-          <param name="min">-1.5708</param>
-          <param name="max">1.5708</param>
+          <param name="min">-6.2832</param>
+          <param name="max">6.2832</param>
         </command_interface>
         <state_interface name="position"/>
@@ -29,9 +27,8 @@
         <state_interface name="effort"/>
       </joint>
-      <!-- Joint 3 -->
-      <joint name="${arm_id}_joint3">
+      <joint name="${arm_id}_elbow_joint">
         <command_interface name="position">
-          <param name="min">-3.14159</param>
-          <param name="max">3.14159</param>
+          <param name="min">-3.1416</param>
+          <param name="max">3.1416</param>
         </command_interface>
         <state_interface name="position"/>
@@ -39,9 +36,8 @@
         <state_interface name="effort"/>
       </joint>
-      <!-- Joint 4 -->
-      <joint name="${arm_id}_joint4">
+      <joint name="${arm_id}_wrist_1_joint">
         <command_interface name="position">
-          <param name="min">-3.14159</param>
-          <param name="max">3.14159</param>
+          <param name="min">-6.2832</param>
+          <param name="max">6.2832</param>
         </command_interface>
         <state_interface name="position"/>
@@ -49,9 +45,8 @@
         <state_interface name="effort"/>
       </joint>
-      <!-- Joint 5 -->
-      <joint name="${arm_id}_joint5">
+      <joint name="${arm_id}_wrist_2_joint">
         <command_interface name="position">
-          <param name="min">-1.5708</param>
-          <param name="max">1.5708</param>
+          <param name="min">-6.2832</param>
+          <param name="max">6.2832</param>
         </command_interface>
         <state_interface name="position"/>
@@ -59,9 +54,8 @@
         <state_interface name="effort"/>
       </joint>
-      <!-- Joint 6 -->
-      <joint name="${arm_id}_joint6">
+      <joint name="${arm_id}_wrist_3_joint">
         <command_interface name="position">
-          <param name="min">-3.14159</param>
-          <param name="max">3.14159</param>
+          <param name="min">-6.2832</param>
+          <param name="max">6.2832</param>
         </command_interface>
         <state_interface name="position"/>
@@ -70,5 +64,4 @@
       </joint>
     </ros2_control>
-    <!-- Gazebo ros2_control plugin -->
     <gazebo>
       <plugin filename="libgazebo_ros2_control.so" name="gazebo_ros2_control">

File: src/teleop_description/urdf/arm_6dof.urdf.xacro (robot description, xacro)
@@ -1,228 +1,226 @@
 <?xml version="1.0"?>
-<robot xmlns:xacro="http://www.ros.org/wiki/xacro" name="arm_6dof">
-  <!-- Arguments -->
-  <xacro:arg name="arm_id" default="master"/>
-  <xacro:arg name="initial_positions_file" default="initial_positions.yaml"/>
-  <!-- Parameters -->
-  <xacro:property name="arm_id" value="$(arg arm_id)" />
-  <xacro:property name="PI" value="3.14159265359"/>
-  <!-- Materials -->
-  <material name="black">
-    <color rgba="0.0 0.0 0.0 1.0"/>
-  </material>
-  <material name="blue">
-    <color rgba="0.0 0.0 0.8 1.0"/>
-  </material>
-  <material name="green">
-    <color rgba="0.0 0.8 0.0 1.0"/>
-  </material>
-  <!-- Base Link -->
-  <link name="${arm_id}_base_link">
-    <visual>
-      <geometry>
-        <cylinder radius="0.05" length="0.1"/>
-      </geometry>
-      <origin xyz="0 0 0.05" rpy="0 0 0"/>
-      <material name="black"/>
-    </visual>
-    <collision>
-      <geometry>
-        <cylinder radius="0.05" length="0.1"/>
-      </geometry>
-      <origin xyz="0 0 0.05" rpy="0 0 0"/>
-    </collision>
-    <inertial>
-      <mass value="1.0"/>
-      <inertia ixx="0.01" ixy="0.0" ixz="0.0" iyy="0.01" iyz="0.0" izz="0.01"/>
-    </inertial>
-  </link>
-  <!-- Link 1 -->
-  <link name="${arm_id}_link1">
-    <visual>
-      <geometry>
-        <cylinder radius="0.04" length="0.3"/>
-      </geometry>
+<robot xmlns:xacro="http://www.ros.org/wiki/xacro">
+  <!-- Define a macro for 6-DOF arm that can be instantiated with different prefixes -->
+  <xacro:macro name="arm_6dof" params="prefix">
+    <xacro:property name="PI" value="3.14159265359"/>
+    <!-- Materials -->
+    <material name="${prefix}_black">
+      <color rgba="0.0 0.0 0.0 1.0"/>
+    </material>
+    <material name="${prefix}_blue">
+      <color rgba="0.0 0.0 0.8 1.0"/>
+    </material>
+    <material name="${prefix}_green">
+      <color rgba="0.0 0.8 0.0 1.0"/>
+    </material>
+    <!-- Base Link -->
+    <link name="${prefix}_base_link">
+      <visual>
+        <geometry>
+          <cylinder radius="0.05" length="0.1"/>
+        </geometry>
+        <origin xyz="0 0 0.05" rpy="0 0 0"/>
+        <material name="${prefix}_black"/>
+      </visual>
+      <collision>
+        <geometry>
+          <cylinder radius="0.05" length="0.1"/>
+        </geometry>
+        <origin xyz="0 0 0.05" rpy="0 0 0"/>
+      </collision>
+      <inertial>
+        <mass value="1.0"/>
+        <inertia ixx="0.01" ixy="0.0" ixz="0.0" iyy="0.01" iyz="0.0" izz="0.01"/>
+      </inertial>
+    </link>
+    <!-- Link 1 -->
+    <link name="${prefix}_link1">
+      <visual>
+        <geometry>
+          <cylinder radius="0.04" length="0.3"/>
+        </geometry>
+        <origin xyz="0 0 0.15" rpy="0 0 0"/>
+        <material name="${prefix}_blue"/>
+      </visual>
+      <collision>
+        <geometry>
+          <cylinder radius="0.04" length="0.3"/>
+        </geometry>
+        <origin xyz="0 0 0.15" rpy="0 0 0"/>
+      </collision>
+      <inertial>
+        <mass value="0.5"/>
+        <inertia ixx="0.005" ixy="0.0" ixz="0.0" iyy="0.005" iyz="0.0" izz="0.001"/>
+      </inertial>
+    </link>
+    <!-- Joint 1 -->
+    <joint name="${prefix}_joint1" type="revolute">
+      <parent link="${prefix}_base_link"/>
+      <child link="${prefix}_link1"/>
+      <origin xyz="0 0 0.1" rpy="0 0 0"/>
+      <axis xyz="0 0 1"/>
+      <limit effort="100.0" lower="${-PI}" upper="${PI}" velocity="2.0"/>
+      <dynamics damping="0.5" friction="0.5"/>
+    </joint>
+    <!-- Link 2 -->
+    <link name="${prefix}_link2">
+      <visual>
+        <geometry>
+          <cylinder radius="0.035" length="0.25"/>
+        </geometry>
+        <origin xyz="0 0 0.125" rpy="0 0 0"/>
+        <material name="${prefix}_green"/>
+      </visual>
+      <collision>
+        <geometry>
+          <cylinder radius="0.035" length="0.25"/>
+        </geometry>
+        <origin xyz="0 0 0.125" rpy="0 0 0"/>
+      </collision>
+      <inertial>
+        <mass value="0.4"/>
+        <inertia ixx="0.003" ixy="0.0" ixz="0.0" iyy="0.003" iyz="0.0" izz="0.001"/>
+      </inertial>
+    </link>
+    <!-- Joint 2 -->
+    <joint name="${prefix}_joint2" type="revolute">
+      <parent link="${prefix}_link1"/>
+      <child link="${prefix}_link2"/>
+      <origin xyz="0 0 0.3" rpy="0 0 0"/>
+      <axis xyz="0 1 0"/>
+      <limit effort="100.0" lower="${-PI/2}" upper="${PI/2}" velocity="2.0"/>
+      <dynamics damping="0.5" friction="0.5"/>
+    </joint>
+    <!-- Link 3 -->
+    <link name="${prefix}_link3">
+      <visual>
+        <geometry>
+          <cylinder radius="0.03" length="0.25"/>
+        </geometry>
+        <origin xyz="0 0 0.125" rpy="0 0 0"/>
+        <material name="${prefix}_blue"/>
+      </visual>
+      <collision>
+        <geometry>
+          <cylinder radius="0.03" length="0.25"/>
+        </geometry>
+        <origin xyz="0 0 0.125" rpy="0 0 0"/>
+      </collision>
+      <inertial>
+        <mass value="0.3"/>
+        <inertia ixx="0.002" ixy="0.0" ixz="0.0" iyy="0.002" iyz="0.0" izz="0.0005"/>
+      </inertial>
+    </link>
+    <!-- Joint 3 -->
+    <joint name="${prefix}_joint3" type="revolute">
+      <parent link="${prefix}_link2"/>
+      <child link="${prefix}_link3"/>
+      <origin xyz="0 0 0.25" rpy="0 0 0"/>
+      <axis xyz="0 1 0"/>
+      <limit effort="50.0" lower="${-PI}" upper="${PI}" velocity="2.0"/>
+      <dynamics damping="0.3" friction="0.3"/>
+    </joint>
+    <!-- Link 4 -->
+    <link name="${prefix}_link4">
+      <visual>
+        <geometry>
+          <cylinder radius="0.025" length="0.15"/>
+        </geometry>
+        <origin xyz="0 0 0.075" rpy="0 0 0"/>
+        <material name="${prefix}_green"/>
+      </visual>
+      <collision>
+        <geometry>
+          <cylinder radius="0.025" length="0.15"/>
+        </geometry>
+        <origin xyz="0 0 0.075" rpy="0 0 0"/>
+      </collision>
+      <inertial>
+        <mass value="0.2"/>
+        <inertia ixx="0.001" ixy="0.0" ixz="0.0" iyy="0.001" iyz="0.0" izz="0.0003"/>
+      </inertial>
+    </link>
+    <!-- Joint 4 -->
+    <joint name="${prefix}_joint4" type="revolute">
+      <parent link="${prefix}_link3"/>
+      <child link="${prefix}_link4"/>
+      <origin xyz="0 0 0.25" rpy="0 0 0"/>
+      <axis xyz="0 0 1"/>
+      <limit effort="25.0" lower="${-PI}" upper="${PI}" velocity="3.0"/>
+      <dynamics damping="0.2" friction="0.2"/>
+    </joint>
+    <!-- Link 5 -->
+    <link name="${prefix}_link5">
+      <visual>
+        <geometry>
+          <cylinder radius="0.02" length="0.1"/>
+        </geometry>
+        <origin xyz="0 0 0.05" rpy="0 0 0"/>
+        <material name="${prefix}_blue"/>
+      </visual>
+      <collision>
+        <geometry>
+          <cylinder radius="0.02" length="0.1"/>
+        </geometry>
+        <origin xyz="0 0 0.05" rpy="0 0 0"/>
+      </collision>
+      <inertial>
+        <mass value="0.15"/>
+        <inertia ixx="0.0005" ixy="0.0" ixz="0.0" iyy="0.0005" iyz="0.0" izz="0.0002"/>
+      </inertial>
+    </link>
+    <!-- Joint 5 -->
+    <joint name="${prefix}_joint5" type="revolute">
+      <parent link="${prefix}_link4"/>
+      <child link="${prefix}_link5"/>
       <origin xyz="0 0 0.15" rpy="0 0 0"/>
-      <material name="blue"/>
-    </visual>
-    <collision>
-      <geometry>
-        <cylinder radius="0.04" length="0.3"/>
-      </geometry>
-      <origin xyz="0 0 0.15" rpy="0 0 0"/>
-    </collision>
-    <inertial>
-      <mass value="0.5"/>
-      <inertia ixx="0.005" ixy="0.0" ixz="0.0" iyy="0.005" iyz="0.0" izz="0.001"/>
-    </inertial>
-  </link>
-  <!-- Joint 1 (Base rotation - Z axis) -->
-  <joint name="${arm_id}_joint1" type="revolute">
-    <parent link="${arm_id}_base_link"/>
-    <child link="${arm_id}_link1"/>
-    <origin xyz="0 0 0.1" rpy="0 0 0"/>
-    <axis xyz="0 0 1"/>
-    <limit effort="100.0" lower="${-PI}" upper="${PI}" velocity="2.0"/>
-    <dynamics damping="0.5" friction="0.5"/>
-  </joint>
-  <!-- Link 2 -->
-  <link name="${arm_id}_link2">
-    <visual>
-      <geometry>
-        <cylinder radius="0.035" length="0.25"/>
-      </geometry>
-      <origin xyz="0 0 0.125" rpy="0 0 0"/>
-      <material name="green"/>
-    </visual>
-    <collision>
-      <geometry>
-        <cylinder radius="0.035" length="0.25"/>
-      </geometry>
-      <origin xyz="0 0 0.125" rpy="0 0 0"/>
-    </collision>
-    <inertial>
-      <mass value="0.4"/>
-      <inertia ixx="0.003" ixy="0.0" ixz="0.0" iyy="0.003" iyz="0.0" izz="0.001"/>
-    </inertial>
-  </link>
-  <!-- Joint 2 (Shoulder - Y axis) -->
-  <joint name="${arm_id}_joint2" type="revolute">
-    <parent link="${arm_id}_link1"/>
-    <child link="${arm_id}_link2"/>
-    <origin xyz="0 0 0.3" rpy="0 0 0"/>
-    <axis xyz="0 1 0"/>
-    <limit effort="100.0" lower="${-PI/2}" upper="${PI/2}" velocity="2.0"/>
-    <dynamics damping="0.5" friction="0.5"/>
-  </joint>
-  <!-- Link 3 -->
-  <link name="${arm_id}_link3">
-    <visual>
-      <geometry>
-        <cylinder radius="0.03" length="0.25"/>
-      </geometry>
-      <origin xyz="0 0 0.125" rpy="0 0 0"/>
-      <material name="blue"/>
-    </visual>
-    <collision>
-      <geometry>
-        <cylinder radius="0.03" length="0.25"/>
-      </geometry>
-      <origin xyz="0 0 0.125" rpy="0 0 0"/>
-    </collision>
-    <inertial>
-      <mass value="0.3"/>
-      <inertia ixx="0.002" ixy="0.0" ixz="0.0" iyy="0.002" iyz="0.0" izz="0.0005"/>
-    </inertial>
-  </link>
-  <!-- Joint 3 (Elbow - Y axis) -->
-  <joint name="${arm_id}_joint3" type="revolute">
-    <parent link="${arm_id}_link2"/>
-    <child link="${arm_id}_link3"/>
-    <origin xyz="0 0 0.25" rpy="0 0 0"/>
-    <axis xyz="0 1 0"/>
-    <limit effort="50.0" lower="${-PI}" upper="${PI}" velocity="2.0"/>
-    <dynamics damping="0.3" friction="0.3"/>
-  </joint>
-  <!-- Link 4 -->
-  <link name="${arm_id}_link4">
-    <visual>
-      <geometry>
-        <cylinder radius="0.025" length="0.15"/>
-      </geometry>
-      <origin xyz="0 0 0.075" rpy="0 0 0"/>
-      <material name="green"/>
-    </visual>
-    <collision>
-      <geometry>
-        <cylinder radius="0.025" length="0.15"/>
-      </geometry>
-      <origin xyz="0 0 0.075" rpy="0 0 0"/>
-    </collision>
-    <inertial>
-      <mass value="0.2"/>
-      <inertia ixx="0.001" ixy="0.0" ixz="0.0" iyy="0.001" iyz="0.0" izz="0.0003"/>
-    </inertial>
-  </link>
-  <!-- Joint 4 (Wrist roll - Z axis) -->
-  <joint name="${arm_id}_joint4" type="revolute">
-    <parent link="${arm_id}_link3"/>
-    <child link="${arm_id}_link4"/>
-    <origin xyz="0 0 0.25" rpy="0 0 0"/>
-    <axis xyz="0 0 1"/>
-    <limit effort="25.0" lower="${-PI}" upper="${PI}" velocity="3.0"/>
-    <dynamics damping="0.2" friction="0.2"/>
-  </joint>
-  <!-- Link 5 -->
-  <link name="${arm_id}_link5">
-    <visual>
-      <geometry>
-        <cylinder radius="0.02" length="0.1"/>
-      </geometry>
-      <origin xyz="0 0 0.05" rpy="0 0 0"/>
-      <material name="blue"/>
-    </visual>
-    <collision>
-      <geometry>
-        <cylinder radius="0.02" length="0.1"/>
-      </geometry>
-      <origin xyz="0 0 0.05" rpy="0 0 0"/>
-    </collision>
-    <inertial>
-      <mass value="0.15"/>
-      <inertia ixx="0.0005" ixy="0.0" ixz="0.0" iyy="0.0005" iyz="0.0" izz="0.0002"/>
-    </inertial>
-  </link>
-  <!-- Joint 5 (Wrist pitch - Y axis) -->
-  <joint name="${arm_id}_joint5" type="revolute">
-    <parent link="${arm_id}_link4"/>
-    <child link="${arm_id}_link5"/>
-    <origin xyz="0 0 0.15" rpy="0 0 0"/>
-    <axis xyz="0 1 0"/>
-    <limit effort="25.0" lower="${-PI/2}" upper="${PI/2}" velocity="3.0"/>
-    <dynamics damping="0.2" friction="0.2"/>
-  </joint>
-  <!-- Link 6 (End-effector) -->
-  <link name="${arm_id}_link6">
-    <visual>
-      <geometry>
-        <cylinder radius="0.015" length="0.08"/>
-      </geometry>
-      <origin xyz="0 0 0.04" rpy="0 0 0"/>
-      <material name="green"/>
-    </visual>
-    <collision>
-      <geometry>
-        <cylinder radius="0.015" length="0.08"/>
-      </geometry>
-      <origin xyz="0 0 0.04" rpy="0 0 0"/>
-    </collision>
-    <inertial>
-      <mass value="0.1"/>
-      <inertia ixx="0.0003" ixy="0.0" ixz="0.0" iyy="0.0003" iyz="0.0" izz="0.0001"/>
-    </inertial>
-  </link>
-  <!-- Joint 6 (Wrist yaw - Z axis) -->
-  <joint name="${arm_id}_joint6" type="revolute">
-    <parent link="${arm_id}_link5"/>
-    <child link="${arm_id}_link6"/>
-    <origin xyz="0 0 0.1" rpy="0 0 0"/>
-    <axis xyz="0 0 1"/>
-    <limit effort="10.0" lower="${-PI}" upper="${PI}" velocity="3.0"/>
-    <dynamics damping="0.1" friction="0.1"/>
-  </joint>
-  <!-- End-effector link (for tool center point) -->
-  <link name="${arm_id}_ee_link">
-    <visual>
-      <geometry>
-        <sphere radius="0.01"/>
-      </geometry>
-      <material name="black"/>
-    </visual>
-  </link>
-  <!-- End-effector joint -->
-  <joint name="${arm_id}_ee_joint" type="fixed">
-    <parent link="${arm_id}_link6"/>
-    <child link="${arm_id}_ee_link"/>
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
File: src/teleop_description/urdf/complete_system.urdf.xacro (robot description, xacro)
@@ -1,25 +1,37 @@
 <?xml version="1.0"?>
 <robot xmlns:xacro="http://www.ros.org/wiki/xacro" name="teleoperation_system">
-  <!-- Include arm macros -->
-  <xacro:include filename="$(find teleop_description)/urdf/arm_6dof.urdf.xacro"/>
-  <xacro:include filename="$(find teleop_description)/urdf/arm_6dof.ros2_control.xacro"/>
+  <!-- Include UR macro and combined ros2_control -->
+  <xacro:include filename="$(find ur_description)/urdf/ur_macro.xacro"/>
+  <xacro:include filename="$(find teleop_description)/urdf/combined.ros2_control.xacro"/>
+  <!-- UR5 Configuration files -->
+  <xacro:arg name="joint_limit_params" default="$(find ur_description)/config/ur5/joint_limits.yaml"/>
+  <xacro:arg name="kinematics_params" default="$(find ur_description)/config/ur5/default_kinematics.yaml"/>
+  <xacro:arg name="physical_params" default="$(find ur_description)/config/ur5/physical_parameters.yaml"/>
+  <xacro:arg name="visual_params" default="$(find ur_description)/config/ur5/visual_parameters.yaml"/>
   <!-- World link -->
   <link name="world"/>
-  <!-- Master Arm -->
-  <xacro:property name="master_arm_id" value="master"/>
-  <joint name="world_to_master" type="fixed">
-    <parent link="world"/>
-    <child link="master_base_link"/>
-    <origin xyz="-0.5 0 0" rpy="0 0 0"/>
-  </joint>
-  <!-- Slave Arm -->
-  <xacro:property name="slave_arm_id" value="slave"/>
-  <joint name="world_to_slave" type="fixed">
-    <parent link="world"/>
-    <child link="slave_base_link"/>
-    <origin xyz="0.5 0 0" rpy="0 0 0"/>
-  </joint>
-  <!-- Include ros2_control for both arms -->
-  <xacro:arm_6dof_ros2_control arm_id="master" use_sim="true"/>
-  <xacro:arm_6dof_ros2_control arm_id="slave" use_sim="true"/>
+  <!-- Master Arm (UR5) - Default zero position -->
+  <xacro:ur_robot
+    name="master"
+    tf_prefix="master_"
+    parent="world"
+    joint_limits_parameters_file="$(arg joint_limit_params)"
+    kinematics_parameters_file="$(arg kinematics_params)"
+    physical_parameters_file="$(arg physical_params)"
+    visual_parameters_file="$(arg visual_params)">
+    <origin xyz="-0.5 0 0.1" rpy="0 0 0"/>
+  </xacro:ur_robot>
+  <!-- Slave Arm (UR5) - Default zero position -->
+  <xacro:ur_robot
+    name="slave"
+    tf_prefix="slave_"
+    parent="world"
+    joint_limits_parameters_file="$(arg joint_limit_params)"
+    kinematics_parameters_file="$(arg kinematics_params)"
+    physical_parameters_file="$(arg physical_params)"
+    visual_parameters_file="$(arg visual_params)">
+    <origin xyz="0.5 0 0.1" rpy="0 0 0"/>
+  </xacro:ur_robot>
+  <!-- SINGLE combined ros2_control for both arms -->
+  <xacro:combined_ros2_control use_sim="true"/>
 </robot>
